File: motor interfacing.sch (EAGLE design)
At the start: 15 parts

Commit message: Update motor interfacing board
Parts:
- added PYRO: JST-XH-02-PIN-LONG-PAD, Rembrandt Electronics - JST XH Connectors v1-0:JST-XH-02-PIN-LONG-PAD
- added Q1: 60V/32A/35mΩ, SparkFun-DiscreteSemi:MOSFET-NCH-FQP30N06L
- CAN1, CAN2, CAN3: device SparkFun-IC-Comms:MCP2551 -> elm:MCP2551
- R1, R2, R3: device SparkFun-Resistors:20KOHM-0603-1/10W-1% -> SparkFun-Resistors:1KOHM-HORIZ-1/4W-5%
Connections:
- new net N$10: PYRO-1.S, Q1.S
- new net PG0: CN9.29, Q1.G
- net GND: now also PYRO-2.S
- net VCC: now also Q1.D
Other:
- moved on the sheet: CAN1_DB9, CAN2_DB9, CAN3_DB9, D2, R1, R2, R3
